File: Technik-MIT/Technik-MIT.kicad_pcb (KiCad board)
At the start: 2 copper layers, 15.2 x 7 mm, 127 parts, among them J1 USB_C_Receptacle_USB2.0, SW1 SW_Push, SW10 SW_Push, SW11 SW_Push, SW12 SW_Push, SW13 SW_Push, SW14 SW_Push, SW15 SW_Push, SW16 SW_Push, SW17 SW_Push, SW18 SW_Push, SW19 SW_Push, SW2 SW_Push, SW20 SW_Push, SW21 SW_Push, SW22 SW_Push, SW23 SW_Push, SW24 SW_Push, SW25 SW_Push, SW26 SW_Push, SW27 SW_Push, SW28 SW_Push, SW29 SW_Push, SW3 SW_Push, SW30 SW_Push, SW31 SW_Push, SW32 SW_Push, SW33 SW_Push, SW34 SW_Push, SW35 SW_Push, SW36 SW_Push, SW37 SW_Push, SW38 SW_Push, SW39 SW_Push, SW4 SW_Push, SW40 SW_Push, SW41 SW_Push, SW42 SW_Push, SW43 SW_Push, SW44 SW_Push, SW45 SW_Push, SW46 SW_Push, SW47 SW_Push, SW48 SW_Push, SW49 RESET, SW5 SW_Push, SW50 SW_Push, SW6 SW_Push, SW7 SW_Push, SW8 SW_Push, SW9 SW_Push, U1 USBLC6-2SC6, U2 TVS0500DRV, U3 NCP1117-3.3_SOT223, U4 W25Q32JVSS, U5 RP2040, Y1 12MHz

Commit message: Working on PCB
Parts:
- U3: value NCP1117-3.3_SOT223 -> AP2127N-3.3; footprint Package_TO_SOT_SMD:SOT-223-3_TabPin2 -> Package_TO_SOT_SMD:SOT-23
- moved SW49 200.0 mm to (42.6, 71.4)
- moved U1 108.0 mm to (233.6, 42.4), turned to -90 degrees
- moved U2 106.6 mm to (238.4, 39.9)
- moved U3 85.7 mm to (228.8, 53.8), turned to 90 degrees
- moved C8 83.7 mm to (269.6, 44.2), turned to -135 degrees
- moved R2 80.0 mm to (236.4, 39.8), turned to 90 degrees
- moved R1 78.5 mm to (230.8, 39.6), turned to 90 degrees
- moved C3 73.9 mm to (278.2, 60.9)
- moved C4 73.9 mm to (278.2, 62.9)
- moved C5 73.9 mm to (278.2, 64.8)
- moved C6 73.9 mm to (278.2, 66.8)
- moved R3 73.9 mm to (281.1, 60.9)
- moved R6 73.9 mm to (281.1, 66.9)
- moved C1 73.9 mm to (278.2, 56.9)
- moved C2 73.9 mm to (278.2, 58.9)
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Routing:
- net +3V3: track 0.00 -> 37.8 mm
- net /USB_D+: track 0.00 -> 31.3 mm
- net /USB_D-: track 0.00 -> 30.7 mm
- net VBUS: track 0.00 -> 30.1 mm, vias 0 -> 2
- net /QSPI_SD3: track 0.00 -> 30.0 mm
- net /QSPI_SCLK: track 0.00 -> 26.5 mm
- net /QSPI_SD0: track 0.00 -> 22.3 mm
- net /QSPI_SD2: track 0.00 -> 14.4 mm
- net /QSPI_SD1: track 0.00 -> 13.8 mm
- net /QSPI_SS: track 0.00 -> 12.7 mm
- net Net-(J1-D+-PadA6): track 0.00 -> 10.3 mm, vias 0 -> 2
- net Net-(J1-D--PadA7): track 0.00 -> 9.96 mm, vias 0 -> 2
- net Net-(J1-CC1): track 0.00 -> 2.96 mm
- net Net-(J1-CC2): track 0.00 -> 2.79 mm
- net Net-(U5-USB_DM): track 0.00 -> 1.84 mm
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
Commit message: Working on PCB
Parts:
- DIP1: footprint Button_Switch_SMD:SW_DIP_SPSTx01_Slide_6.7x4.1mm_W8.61mm_P2.54mm_LowProfile -> Button_Switch_SMD:SW_SPDT_PCM12
- Y1: value 12MHz -> Crystal_GND24; footprint Crystal:Crystal_SMD_7050-4Pin_7.0x5.0mm -> Crystal:Crystal_SMD_3225-4Pin_3.2x2.5mm
- moved DIP1 230.1 mm to (27.2, 55.0), turned to 90 degrees
- moved Y1 33.6 mm to (226.2, 77.8), turned to 135 degrees
- moved R5 8.07 mm to (234.9, 69.8), turned to -135 degrees
- moved R4 7.80 mm to (235.7, 70.6), turned to -135 degrees
- moved D2 4.52 mm to (36.9, 56.4)
- turned U5 to 135 degrees
Connections:
- DIP1 pad 1: GND -> Net-(DIP1-A)
- DIP1 pad 2: Net-(DIP1-Pad2) -> GND
- R3 pad 1: Net-(DIP1-Pad2) -> Net-(DIP1-A)
- Y1 pad 1: Net-(C5-Pad2) -> Net-(U5-XIN)
- Y1 pad 2: Net-(U5-XIN) -> GND
- Y1 pad 3: (no net) -> Net-(C5-Pad2)
- Y1 pad 4: (no net) -> GND
Routing:
- net +3V3: track 37.8 -> 20.1 mm
- net /QSPI_SD3: track 30.0 -> 20.2 mm
- net /QSPI_SCLK: track 26.5 -> 17.6 mm
- net /QSPI_SD0: track 22.3 -> 14.0 mm
- net /QSPI_SD2: track 14.4 -> 6.80 mm
- net /QSPI_SD1: track 13.8 -> 6.83 mm
- net /QSPI_SS: track 12.7 -> 7.06 mm
- net Net-(U5-XIN): track 0.00 -> 5.04 mm
- net /USB_D-: track 30.7 -> 29.2 mm

Commit message: Update PCB
Change spacing from MX to Choc
Parts:
- removed the D28 at (151.1, 94.5)
- removed the SW24 at (127.7, 100.0)
- removed the SW28 at (146.7, 100.0)
- added ?: , , F.Cu at (184.5, 79.0)
- added ?: , , F.Cu at (108.5, 79.5)
- added ?: , , F.Cu at (241.5, 59.5)
- added ?: , , F.Cu at (241.5, 95.5)
- added ?: , , F.Cu at (70.5, 95.0)
- added ?: , , F.Cu at (51.5, 59.5)
- C1, C2: value 10u -> 1u
- moved DIP1 234.4 mm to (256.8, 102.5), turned to -90 degrees
- moved C7 49.8 mm to (237.3, 89.2), turned to -135 degrees
- moved C5 49.7 mm to (238.7, 95.0), turned to -45 degrees
- moved C4 49.5 mm to (241.1, 95.6), turned to -135 degrees
- moved R3 48.0 mm to (252.3, 99.4), turned to 135 degrees
- moved R6 46.8 mm to (240.0, 89.4), turned to 45 degrees
- moved C8 44.6 mm to (238.8, 76.5), turned to 90 degrees
- moved C2 42.1 mm to (236.4, 64.0), turned to 0 degrees
- moved C1 40.1 mm to (238.1, 58.7), turned to 0 degrees
- moved C3 38.3 mm to (247.0, 83.2), turned to 0 degrees
- moved C6 36.4 mm to (242.8, 75.4), turned to 90 degrees
- moved C15 28.0 mm to (238.6, 89.3), turned to -135 degrees
- moved C13 26.8 mm to (246.5, 79.0), turned to 90 degrees
- moved Y1 24.8 mm to (239.7, 98.6), turned to 180 degrees
- moved C9 23.3 mm to (235.9, 83.2), turned to 180 degrees
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- renumbered D29 to D28, D30 to D29, D31 to D30, D32 to D31, D33 to D32, D34 to D33, D35 to D34, D36 to D35, D37 to D36, D38 to D37, D39 to D38, D40 to D39, D41 to D40, D42 to D41, D43 to D42, D44 to D43, D45 to D44, D46 to D45, D47 to D46, D48 to D47, SW50 to SW24, SW29 to SW28, SW30 to SW29, SW31 to SW30, SW32 to SW31, SW33 to SW32, SW34 to SW33, SW35 to SW34, SW36 to SW35, SW37 to SW36, SW38 to SW37, SW39 to SW38, SW40 to SW39, SW41 to SW40, SW42 to SW41, SW43 to SW42, SW44 to SW43, SW45 to SW44, SW46 to SW45, SW47 to SW46, SW48 to SW47, SW49 to SW48
Connections:
- SW24 pad 1: Net-(D24-A) -> /COL2
- SW24 pad 2: /COL2 -> Net-(D24-A)
- U5 pad 11: /ROW2 -> unconnected-(U5-GPIO8-Pad11)
- U5 pad 12: /ROW3 -> unconnected-(U5-GPIO9-Pad12)
- U5 pad 13: /ROW4 -> unconnected-(U5-GPIO10-Pad13)
- U5 pad 14: /ROW5 -> unconnected-(U5-GPIO11-Pad14)
- U5 pad 15: /ROW6 -> unconnected-(U5-GPIO12-Pad15)
- U5 pad 16: /ROW7 -> unconnected-(U5-GPIO13-Pad16)
- U5 pad 2: /COL0 -> unconnected-(U5-GPIO0-Pad2)
- U5 pad 29: unconnected-(U5-GPIO18-Pad29) -> /ROW7
- U5 pad 3: /COL1 -> /ROW0
- U5 pad 30: unconnected-(U5-GPIO19-Pad30) -> /ROW3
- U5 pad 31: unconnected-(U5-GPIO20-Pad31) -> /ROW6
- U5 pad 35: unconnected-(U5-GPIO23-Pad35) -> /ROW2
- U5 pad 36: unconnected-(U5-GPIO24-Pad36) -> /COL0
- U5 pad 37: unconnected-(U5-GPIO25-Pad37) -> /COL1
- U5 pad 38: unconnected-(U5-GPIO26_ADC0-Pad38) -> /COL2
- U5 pad 39: unconnected-(U5-GPIO27_ADC1-Pad39) -> /COL3
- U5 pad 4: /COL2 -> /ROW4
- U5 pad 40: unconnected-(U5-GPIO28_ADC2-Pad40) -> /COL4
- U5 pad 41: unconnected-(U5-GPIO29_ADC3-Pad41) -> /COL5
- U5 pad 5: /COL3 -> /ROW1
- U5 pad 6: /COL4 -> /ROW5
- U5 pad 7: /COL5 -> unconnected-(U5-GPIO5-Pad7)
- U5 pad 8: /ROW0 -> unconnected-(U5-GPIO6-Pad8)
- U5 pad 9: /ROW1 -> unconnected-(U5-GPIO7-Pad9)
Routing:
- net /ROW0: track 0.00 -> 255.0 mm, vias 0 -> 9
- net /ROW4: track 0.00 -> 243.4 mm, vias 0 -> 7
- net /ROW1: track 0.00 -> 240.6 mm, vias 0 -> 7
- net /ROW5: track 0.00 -> 220.1 mm, vias 0 -> 6
- net /COL2: track 0.00 -> 111.9 mm
- net /COL0: track 0.00 -> 108.1 mm
- net /COL4: track 0.00 -> 108.0 mm
- net /COL1: track 0.00 -> 108.0 mm
- net /COL5: track 0.00 -> 90.0 mm
- net /COL3: track 0.00 -> 90.0 mm
- net +3V3: track 20.1 -> 62.3 mm
- net +1V1: track 0.00 -> 18.5 mm, vias 0 -> 4
- net Net-(D40-A): track 0.00 -> 15.6 mm
- net Net-(D47-A): track 0.00 -> 14.9 mm
- net Net-(D42-A): track 0.00 -> 14.2 mm
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- added copper zone on B.Cu, net +1V1
- added copper zone on B.Cu, net GND
- added copper zone on F.Cu, net GND
Other:
- board size 15.2 x 7 mm -> 229 x 76.8 mm
